File: hardware/power.kicad_sch (KiCad schematic)
At the start: 36 parts, among them Q4 DMN1150UFB-7B, U3 TI LMR51430YFDDCR, U4 TI LMR51430YFDDCR, U5 TPS2116DRLR, U6 NCV8187AMT180TAG, U7 LP5912-3.3DRVR

Commit message: RP2354A
Other:
- note added: "FPWM version of the LMR51430 for less output ripple at low voltage and more consistency but less efficient"
- note removed: "FPWM version of the LMR51420YFDDCR for less output ripple at low voltage and more consistency but less efficient"
Changed lines of the file:
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@@
 	(text "3.3V 1A MAIN LDO "
 		(exclude_from_sim no)
-		(at 218.186 89.662 0)
+		(at 183.134 81.788 0)
 		(effects
 			(font
@@
 		)
 	)
-	(text "FPWM version of the LMR51420YFDDCR for less output ripple at low voltage and more consistency but less efficient"
+	(text "FPWM version of the LMR51430 for less output ripple at low voltage and more consistency but less efficient"
 		(exclude_from_sim no)
-		(at 72.136 23.876 0)
+		(at 71.12 23.622 0)
 		(effects
 			(font
@@
 		(exclude_from_sim no)
 		(at 21.336 129.54 0)
-		(size 63.5 11.43)
+		(size 63.5 12.1268)
 		(margins 0.9525 0.9525 0.9525 0.9525)
 		(stroke
 			(width 0)
-			(type default)
+			(type solid)
 		)
 		(fill
@@
 		(in_pos_files yes)
 		(dnp no)
-		(fields_autoplaced yes)
 		(property "Reference" "U5"
-			(at 114.3 144.78 0)
+			(at 114.3 162.306 0)
 			(show_name no)
 			(do_not_autoplace no)
@@
 		)
 		(property "Value" "TPS2116DRLR"
-			(at 114.3 147.32 0)
+			(at 114.3 165.1 0)
 			(show_name no)
 			(do_not_autoplace no)
