File: hardware/power.kicad_sch (KiCad schematic)
At the start: 34 parts, among them U3 TI LMR51430YFDDCR, U4 TI LMR51430YFDDCR, U5 TPS2116DRLR, U6 NCV8187AMT180TAG, U7 LP5912-3.3DRVR

Commit message: LED resistors
Also reduced the amount of different resistors for cheaper assembly
Parts:
- removed R34: 200R, Resistor_SMD:R_0201_0603Metric, symbol Device:R
- added R50: 2.4k, Resistor_SMD:R_0201_0603Metric, symbol Device:R
- R30: value 6.34K -> 6.49k; LCSC C100502 -> C2107920; Manufacturer LIZ Elec -> (none)
- R33: value 470R -> 7.5k; LCSC C473464 -> C474437; MPN 0201WMF4700TEE -> (none); Manufacturer UNI-ROYAL -> (none)
- R36: value 30R -> 510R; LCSC C778391 -> C57784; MPN NQ01WMJ0300TEE -> (none); Manufacturer UNI-ROYAL -> (none)
- R40: value 200R -> 2.4k; LCSC C270359 -> C166281; MPN 0201WMF2000TEE -> (none); Manufacturer UNI-ROYAL -> (none)
Connections:
- net +5V_BUCK: now also R50.1
- net at D5.2 (A): now also R50.2
Changed lines of the file:
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@@
 			)
 		)
-		(property "Value" "200R"
+		(property "Value" "2.4k"
 			(at 251.46 55.8799 0)
 			(show_name no)
@@
 			)
 		)
-		(property "LCSC" "C270359"
+		(property "LCSC" "C166281"
 			(at 248.92 54.61 0)
 			(hide yes)
@@
 			)
 		)
-		(property "MPN" "0201WMF2000TEE"
+		(property "MPN" ""
 			(at -8.89 15.24 0)
 			(hide yes)
@@
 			)
 		)
-		(property "Manufacturer" "UNI-ROYAL"
+		(property "Manufacturer" ""
 			(at -8.89 15.24 0)
 			(hide yes)
@@
 	)
 	(symbol
-		(lib_id "Device:R")
-		(at 140.97 88.9 0)
-		(unit 1)
-		(body_style 1)
-		(exclude_from_sim no)
-		(in_bom yes)
-		(on_board yes)
-		(in_pos_files yes)
-		(dnp no)
-		(fields_autoplaced yes)
-		(property "Reference" "R34"
-			(at 143.51 87.6299 0)
-			(show_name no)
-			(do_not_autoplace no)
-			(effects
-				(font
-					(size 1.27 1.27)
-				)
-				(justify left)
-			)
-		)
-		(property "Value" "200R"
-			(at 143.51 90.1699 0)
-			(show_name no)
-			(do_not_autoplace no)
-			(effects
-				(font
-					(size 1.27 1.27)
-				)
-				(justify left)
-			)
-		)
-		(property "Footprint" "Resistor_SMD:R_0201_0603Metric"
-			(at 139.192 88.9 90)
-			(hide yes)
-			(show_name no)
-			(do_not_autoplace no)
-			(effects
-				(font
-					(size 1.27 1.27)
-				)
-			)
-		)
-		(property "Datasheet" ""
-			(at 140.97 88.9 0)
-			(hide yes)
-			(show_name no)
-			(do_not_autoplace no)
-			(effects
-				(font
-					(size 1.27 1.27)
-				)
-			)
-		)
-		(property "Description" "Resistor"
-			(at 140.97 88.9 0)
-			(hide yes)
-			(show_name no)
-			(do_not_autoplace no)
-			(effects
-				(font
-					(size 1.27 1.27)
-				)
-			)
-		)
-		(property "LCSC" "C270359"
-			(at 140.97 88.9 0)
-			(hide yes)
-			(show_name no)
-			(do_not_autoplace no)
-			(effects
-				(font
-					(size 1.27 1.27)
-				)
-			)
-		)
-		(property "MPN" "0201WMF2000TEE"
-			(at 0 0 0)
-			(hide yes)
-			(show_name no)
-			(do_not_autoplace no)
-			(effects
-				(font
-					(size 1.27 1.27)
-				)
-			)
-		)
-		(property "Manufacturer" "UNI-ROYAL"
-			(at 0 0 0)
-			(hide yes)
-			(show_name no)
-			(do_not_autoplace no)
-			(effects
-				(font
-					(size 1.27 1.27)
-				)
-			)
-		)
-		(pin "1"
-		)
-		(pin "2"
-		)
-		(instances
-			(project "OpenFC"
-				(path "/fb88b6f9-ee39-4640-a9d4-04a17ceeac64/f8522f96-c979-41d2-ae00-e5ad899a3161"
-					(reference "R34")
-					(unit 1)
-				)
-			)
-		)
-	)
-	(symbol
 		(lib_id "Device:C")
 		(at 198.12 109.22 0)
@@
 	)
 	(symbol
+		(lib_id "Device:R")
+		(at 140.97 88.9 0)
+		(unit 1)
+		(body_style 1)
+		(exclude_from_sim no)
+		(in_bom yes)
+		(on_board yes)
+		(in_pos_files yes)
+		(dnp no)
+		(fields_autoplaced yes)
+		(property "Reference" "R50"
+			(at 143.51 87.6299 0)
+			(show_name no)
+			(do_not_autoplace no)
+			(effects
+				(font
+					(size 1.27 1.27)
+				)
+				(justify left)
+			)
+		)
+		(property "Value" "2.4k"
+			(at 143.51 90.1699 0)
+			(show_name no)
+			(do_not_autoplace no)
+			(effects
+				(font
+					(size 1.27 1.27)
+				)
+				(justify left)
+			)
+		)
+		(property "Footprint" "Resistor_SMD:R_0201_0603Metric"
+			(at 139.192 88.9 90)
+			(hide yes)
+			(show_name no)
+			(do_not_autoplace no)
+			(effects
+				(font
+					(size 1.27 1.27)
+				)
+			)
+		)
+		(property "Datasheet" ""
+			(at 140.97 88.9 0)
+			(hide yes)
+			(show_name no)
+			(do_not_autoplace no)
+			(effects
+				(font
+					(size 1.27 1.27)
+				)
+			)
+		)
+		(property "Description" "Resistor"
+			(at 140.97 88.9 0)
+			(hide yes)
+			(show_name no)
+			(do_not_autoplace no)
+			(effects
+				(font
+					(size 1.27 1.27)
+				)
+			)
+		)
+		(property "LCSC" "C166281"
+			(at 140.97 88.9 0)
+			(hide yes)
+			(show_name no)
+			(do_not_autoplace no)
+			(effects
+				(font
+					(size 1.27 1.27)
+				)
+			)
+		)
+		(property "MPN" ""
+			(at -116.84 49.53 0)
+			(hide yes)
+			(show_name no)
+			(do_not_autoplace no)
+			(effects
+				(font
+					(size 1.27 1.27)
+				)
+			)
+		)
+		(property "Manufacturer" ""
+			(at -116.84 49.53 0)
+			(hide yes)
+			(show_name no)
+			(do_not_autoplace no)
+			(effects
+				(font
+					(size 1.27 1.27)
+				)
+			)
+		)
+		(pin "1"
+		)
+		(pin "2"
+		)
+		(instances
+			(project "OpenFC"
+				(path "/fb88b6f9-ee39-4640-a9d4-04a17ceeac64/f8522f96-c979-41d2-ae00-e5ad899a3161"
+					(reference "R50")
+					(unit 1)
+				)
+			)
+		)
+	)
+	(symbol
 		(lib_id "power:GND")
 		(at 92.71 104.14 0)
@@
 			)
 		)
-		(property "Value" "6.34K"
+		(property "Value" "6.49k"
 			(at 119.38 58.4199 0)
 			(show_name no)
@@
 			)
 		)
-		(property "LCSC" "C100502"
+		(property "LCSC" "C2107920"
 			(at 116.84 57.15 0)
 			(hide yes)
@@
 			)
 		)
-		(property "Manufacturer" "LIZ Elec"
+		(property "Manufacturer" ""
 			(at 0 0 0)
 			(hide yes)
@@
 			)
 		)
-		(property "Value" "470R"
+		(property "Value" "7.5k"
 			(at 143.51 48.2599 0)
 			(show_name no)
@@
 			)
 		)
-		(property "LCSC" "C473464"
+		(property "LCSC" "C474437"
 			(at 140.97 46.99 0)
 			(hide yes)
@@
 			)
 		)
-		(property "MPN" "0201WMF4700TEE"
+		(property "MPN" ""
 			(at 0 0 0)
 			(hide yes)
@@
 			)
 		)
-		(property "Manufacturer" "UNI-ROYAL"
+		(property "Manufacturer" ""
 			(at 0 0 0)
 			(hide yes)
@@
 			)
 		)
-		(property "Value" "30R"
+		(property "Value" "510R"
 			(at 255.27 106.6799 0)
 			(show_name no)
@@
 			)
 		)
-		(property "LCSC" "C778391"
+		(property "LCSC" "C57784"
 			(at 252.73 105.41 0)
 			(hide yes)
@@
 			)
 		)
-		(property "MPN" "NQ01WMJ0300TEE"
+		(property "MPN" ""
 			(at 0 1.27 0)
 			(hide yes)
@@
 			)
 		)
-		(property "Manufacturer" "UNI-ROYAL"
+		(property "Manufacturer" ""
 			(at 0 1.27 0)
 			(hide yes)
