File: hardware/rp2350a.kicad_sch (KiCad schematic)
At the start: 54 parts, among them Q2 DMN1150UFB-7B, Q3 DMN1150UFB-7B, U1 TS2306A 240GF MSM 9_C2976675, U2 RP2354B_C39843328, X1 XTM25012000JT00351001

Commit message: many tiny improvements
- I/O correctness
- SPI0/SPI1/I2C0 bus corrections
- decoupling of DVDD
- ADC_AVDD as per RPi documents
- removal of SBUS
- connect ESC serial
- remove RUN RC-circuit as per RPi documentation
- some more cleanup for readability
- gyro CLKIN decision
- I2C 4.7k pullup
Parts:
- removed C2, C22: 100n, Capacitor_SMD:C_0201_0603Metric, symbol Device:C
- removed R10, R15: 10k, Resistor_SMD:R_0201_0603Metric, symbol Device:R
- removed R9: 200R, Resistor_SMD:R_0201_0603Metric, symbol Device:R
- added C37: 4.7uF, Capacitor_SMD:C_0402_1005Metric, symbol Device:C
- C21: value 4.7uF -> 100n; footprint Capacitor_SMD:C_0402_1005Metric -> Capacitor_SMD:C_0201_0603Metric; LCSC C23733 -> C76939; MPN CL05A475MP5NRNC -> GRM033R61E104KE14D; Manufacturer Samsung Electro-Mechanics -> Murata Electronics
- R17, R18: value 2.2k -> 4.7k; LCSC C142018 -> C100139; MPN RC0201FR-072K2L -> (none); Manufacturer YAGEO -> (none)
Connections:
- net +1.1V: now also C37.1
- net +3.3V: now also C21.1, R17.2, U2.35 (RUN), U2.59 (ADC_AVDD); no longer R17.1
- net +BATT: now also R1.2; no longer R1.1
- net ADC_VBAT: now also R1.1; no longer R1.2
- net ESC_CURRENT: no longer C14.2
- net EXTERNAL: no longer C16.2
- net GND: now also C14.2, C15.2, C16.2, C37.2; no longer C14.1, C15.1, C16.1
- net RSSI: no longer C15.2
- net at R6.1, U2.49 (GPIO40_ADC0): now also C14.1
- net at R8.1, U2.58 (GPIO47_ADC7): now also C16.1
- net at R7.1, U2.56 (GPIO45_ADC5): now also C15.1
- net I2C_SCL renamed I2C0.SCL
- net I2C0.SCL: now also R17.1; no longer R17.2
- net I2C_SDA renamed I2C0.SDA
- net SBUS: no longer names the net of U2.7 (GPIO9)
- net SPI0.CLKIN renamed GYRO_CLKIN
- no-connect marks 19 -> 23
Other:
- note added: "USB port"
- note added: "i2c for external sensors"
- note added: "vbat sense. 1/11 scale"
- note removed: "USB port with ESD protection"
- note removed: "i2c for barometer and external sensors possibly"
- note removed: "vbat sense. 1/10 scale"
- moved on the sheet: C1, C10, C11, C12, C13, C17, C18, C19, C20, C23, C3, C4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

Commit message: RP2354A
Parts:
- removed C14, C15, C16: 100n, Capacitor_SMD:C_0201_0603Metric, symbol Device:C
- removed C18, C20, C23: 4.7uF, Capacitor_SMD:C_0402_1005Metric, symbol Device:C
- removed L1: AOTA-B201610S3R3-101-T, lib:IND-SMD_L2.0-W1.6_AOTA-B201610S3R3-101-T, symbol lib:AOTA-B201610S3R3-101-T
- removed R11: 10k, Resistor_SMD:R_0201_0603Metric, symbol Device:R
- removed R12, R13, R14: 30R, Resistor_SMD:R_0201_0603Metric, symbol Device:R
- removed R17, R18: 4.7k, Resistor_SMD:R_0201_0603Metric, symbol Device:R
- removed R6, R7, R8: 1k, Resistor_SMD:R_0201_0603Metric, symbol Device:R
- removed U1: TS2306A 240GF MSM 9_C2976675, lib:SW-SMD_4P-L3.0-W2.0-P0.85-LS3.5, symbol lib:TS2306A240GFMSM9_C2976675
- removed U2: RP2354B_C39843328, lib:QFN-80_L10.0-W10.0-P0.40-TL-EP3.4, symbol lib:RP2354B_C39843328
- added C22: 100n, Capacitor_SMD:C_0201_0603Metric, symbol Device:C
- added C44, C45, C46: 4.7uF, Capacitor_SMD:C_0402_1005Metric, symbol Device:C
- added L4: AOTA-B201610S3R3-101-T, lib:IND-SMD_L2.0-W1.6_AOTA-B201610S3R3-101-T, symbol lib:AOTA-B201610S3R3-101-T
- added R15, R24, R37: 30R, Resistor_SMD:R_0201_0603Metric, symbol Device:R
- added R19, R21: 4.7k, Resistor_SMD:R_0201_0603Metric, symbol Device:R
- added R38: 10k, Resistor_SMD:R_0201_0603Metric, symbol Device:R
- added R9: 1k, Resistor_SMD:R_0201_0603Metric, symbol Device:R
- added U10: RP2354A, lib:QFN-60_L7.0-W7.0-P0.40-TL-EP3.4, symbol lib:RP2354A
- added U11: TS2306A 240GF MSM 9_C2976675, lib:SW-SMD_4P-L3.0-W2.0-P0.85-LS3.5, symbol lib:TS2306A240GFMSM9_C2976675
Connections:
- net D+_C is gone; now on net D+: USB1.A6 (DP1), USB1.B6 (DP2)
- net D-_C is gone; now on net D-: USB1.A7 (DN1), USB1.B7 (DN2)
- net +1.1V: now also C46.1, L4.1, U10.23 (DVDD), U10.39 (DVDD), U10.50 (VREG_FB), U10.6 (DVDD)
- net +3.3V: now also C45.1, R15.1, R19.2, R21.2, U10.1 (IOVDD), U10.11 (IOVDD), U10.20 (IOVDD), U10.26 (RUN), U10.30 (IOVDD), U10.38 (IOVDD), U10.44 (ADC_AVDD), U10.45 (IOVDD), U10.49 (VREG_VIN), U10.53 (USB_OTP_VDD), U10.54 (QSPI_IOVDD)
- net 10V_ENABLE: now also U10.42 (GPIO28_ADC2)
- net ADC_VBAT: now also U10.40 (GPIO26_ADC0)
- net BEEPER: now also U10.9 (GPIO6)
- net D+: now also R37.2
- net D-: now also R24.1
- net ESC_CURRENT: now also R9.1
- net FLASH_CS: now also U10.17 (GPIO13)
- net GND: now also C22.2, C44.2, C45.2, C46.2, U10.47 (VREG_PGND), U10.61 (EP), U11.1
- net GYRO_CS: now also U10.33 (GPIO21)
- net GYRO_INT: now also U10.28 (GPIO17)
- net I2C0.SCL: now also R19.1, U10.7 (GPIO4)
- net I2C0.SDA: now also R21.1, U10.8 (GPIO5)
- net LED0: now also U10.43 (GPIO29_ADC3)
- net LED_STRIP_L: now also U10.10 (GPIO7)
- net MOTOR1: now also U10.37 (GPIO25)
- net MOTOR2: now also U10.36 (GPIO24)
- net MOTOR3: now also U10.35 (GPIO23)
- net MOTOR4: now also U10.34 (GPIO22)
- net OSD_EN: now also U10.19 (GPIO15)
- net OSD_SYNC: now also U10.27 (GPIO16)
- net OSD_W: now also U10.18 (GPIO14)
- net PIOUART0_RX: now also U10.13 (GPIO9)
- net PIOUART0_TX: now also U10.12 (GPIO8)
- net SPI0.MISO: now also U10.32 (GPIO20)
- net SPI0.MOSI: now also U10.31 (GPIO19)
- net SPI0.SCK: now also U10.29 (GPIO18)
- net SPI1.MISO: now also U10.16 (GPIO12)
- net SPI1.MOSI: now also U10.15 (GPIO11)
- net SPI1.SCK: now also U10.14 (GPIO10)
- net UART0_RX: now also U10.3 (GPIO1)
- net UART0_TX: now also U10.2 (GPIO0)
- net UART1_RX: now also U10.5 (GPIO3)
- net UART1_TX: now also U10.4 (GPIO2)
- net XIN: now also U10.21 (XIN)
- net XOUT: now also U10.22 (XOUT)
- new net: R38.1, U11.2
- new net: R38.2, U10.60 (QSPI_SS)
- new net: R24.2, U10.51 (USB_DM)
- new net: C44.1, R15.2, U10.46 (VREG_AVDD)
- new net: L4.2, U10.48 (VREG_LX)
- new net: R37.1, U10.52 (USB_DP)
- new net ESC_CURR: C22.1, R9.2, U10.41 (GPIO27_ADC1)
- no-connect marks 23 -> 9
Other:
- note added: "RP2350 1.1V DC-DC SMPS Follow datasheet guidance on component placement"
- note added: "RP2354A: Smaller variant with integrated flash (2MB)"
- note added: "gyro SPI"
- note removed: "1.1V SMPS by RP datasheet inductor polarity important"
- note removed: "RC lowpass filters on ADC and VREG like Pico datasheet"
- note removed: "RP2350 1.8V DC-DC SMPS Follow datasheet guidance on component placement"
- note removed: "RP2354B: Larger variant with integrated flash (2MB) and more GPIO"
- note removed: "for external (extra)"
- note removed: "gyro SPI line, seperate from blackbox"
- moved on the sheet: C1, C10, C11, C12, C13, C17, C19, C21, C3, C37, C4, C5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
