File: hardware/rp2350a.kicad_sch (KiCad schematic)
At the start: 54 parts, among them Q2 DMN1150UFB-7B, Q3 DMN1150UFB-7B, U1 TS2306A 240GF MSM 9_C2976675, U2 RP2354B_C39843328, X1 XTM25012000JT00351001

Commit message: Rev 2 (RP2354A): finalize design, update docs, clean repo (#5)
* docs(readme): add analog OSD BOM to Rev 2 change list

Document OSD debugging findings and component changes as a new
Analog OSD section in the Rev 2 Change List:
- HW-12: U19 op-amp TLV9061IDPWR -> COS8051SOT (175MHz video-grade RRIO)
- HW-13: output front-end add AC-couple + DC-restore, power U19 from +5V
- HW-14: U20 comparator TLV3201AIDBVR -> TLV7031DPWR (push-pull, X2SON, ~75% smaller)
- HW-15: add OSD_EN select pull-down (datasheet-required, defaults to pass-through)
- U18 / D9 verified correct, no change; OSD GPIO mapping noted (PA4/5/6)

Also fix HW-11 beeper GPIO: GPIO6 -> GPIO7 (GPIO6 is OSD_SYNC per netlist).

Co-Authored-By: Claude Opus 4.8 (1M context) <noreply@anthropic.com>

* many tiny improvements

- I/O correctness
- SPI0/SPI1/I2C0 bus corrections
- decoupling of DVDD
- ADC_AVDD as per RPi documents
- removal of SBUS
- connect ESC serial
- remove RUN RC-circuit as per RPi documentation
- some more cleanup for readability
- gyro CLKIN decision
- I2C 4.7k pullup

* RP2354A

* piu1

* switch spi

* Update OpenFC.kicad_pcb

* routex2

* some minor tweaks

- remove some unnecessary resistors
- slightly higher 10V rail to account for voltage drop
- some cleanup
- simpler PG 1.8V circuit

* Update imu.kicad_sch

* LED resistors

Also reduced the amount of different resistors for cheaper assembly

* Delete leds.kicad_sch

* remove some unneeded decoupling caps from RP2350

* update MOSFET part numbers

* OSD

* ROUTE

* clean libs

* details

* led names

* Clean routing

* docs: rewrite README + CLAUDE.md for finalized Rev 2 (RP2354A)

Rev 2 is a substantial redesign that the docs no longer matched. Updated
both to the actual schematic, verified from the current netlist:

- MCU: RP2354B (QFN-80, GPIO0-47) -> RP2354A (QFN-60, GPIO0-29). Full GPIO
  map re-derived from the netlist + QFN-60 pinout; all 30 GPIO documented.
- IMU moved to SPI1, microSD to SPI0; ref designators re-annotated
  (op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
Parts:
- removed C14, C15, C16, C17, C19, C2: 100n, Capacitor_SMD:C_0201_0603Metric, symbol Device:C
- removed C18, C20, C21, C23: 4.7uF, Capacitor_SMD:C_0402_1005Metric, symbol Device:C
- removed L1: AOTA-B201610S3R3-101-T, lib:IND-SMD_L2.0-W1.6_AOTA-B201610S3R3-101-T, symbol lib:AOTA-B201610S3R3-101-T
- removed Q2, Q3: DMN1150UFB-7B, lib:DFN-3L_L1.0-W0.6-P0.65-BR, symbol lib:DMN1150UFB-7B
- removed R10, R11: 10k, Resistor_SMD:R_0201_0603Metric, symbol Device:R
- removed R12, R13, R14, R16: 30R, Resistor_SMD:R_0201_0603Metric, symbol Device:R
- removed R17, R18, R22, R25: 2.2k, Resistor_SMD:R_0201_0603Metric, symbol Device:R
- removed R20, R8: 1k, Resistor_SMD:R_0201_0603Metric, symbol Device:R
- removed R26: 200R, Resistor_SMD:R_0201_0603Metric, symbol Device:R
- removed U1: TS2306A 240GF MSM 9_C2976675, lib:SW-SMD_4P-L3.0-W2.0-P0.85-LS3.5, symbol lib:TS2306A240GFMSM9_C2976675
- removed U2: RP2354B_C39843328, lib:QFN-80_L10.0-W10.0-P0.40-TL-EP3.4, symbol lib:RP2354B_C39843328
- added C37, C44, C45, C46: 4.7uF, Capacitor_SMD:C_0402_1005Metric, symbol Device:C
- added L4: AOTA-B201610S3R3-101-T, lib:IND-SMD_L2.0-W1.6_AOTA-B201610S3R3-101-T, symbol lib:AOTA-B201610S3R3-101-T
- added Q5, Q6: AP1606, lib:DFN-3L_L1.0-W0.6-P0.65-BR, symbol lib:DMN1150UFB-7B
- added R24, R37: 30R, Resistor_SMD:R_0201_0603Metric, symbol Device:R
- added R38: 10k, Resistor_SMD:R_0201_0603Metric, symbol Device:R
- added R51: 2.4k, Resistor_SMD:R_0201_0603Metric, symbol Device:R
- added R52, R53: 75R, Resistor_SMD:R_0201_0603Metric, symbol Device:R
- added U10: RP2354A, lib:QFN-60_L7.0-W7.0-P0.40-TL-EP3.4, symbol lib:RP2354A
- added U11: TS2306A 240GF MSM 9_C2976675, lib:SW-SMD_4P-L3.0-W2.0-P0.85-LS3.5, symbol lib:TS2306A240GFMSM9_C2976675
- R15: value 10k -> 30R; LCSC C106225 -> C778391; MPN RC0201FR-0710KL -> NQ01WMJ0300TEE; Manufacturer YAGEO -> UNI-ROYAL
- R6, R7: value 1k -> 5.1k; LCSC C270365 -> C270344; MPN 0201WMF1001TEE -> 0201WMF5101TEE
- R9: value 200R -> 1k; LCSC C270359 -> C270365; MPN 0201WMF2000TEE -> 0201WMF1001TEE
Connections:
- net D+_C is gone; now on net D+: USB1.A6 (DP1), USB1.B6 (DP2)
- net D-_C is gone; now on net D-: USB1.A7 (DN1), USB1.B7 (DN2)
- net +1.1V: now also C37.1, C46.1, L4.1, U10.23 (DVDD), U10.39 (DVDD), U10.50 (VREG_FB), U10.6 (DVDD)
- net +3.3V: now also R15.1, R6.1, R7.1, C45.1, U10.1 (IOVDD), U10.11 (IOVDD), U10.20 (IOVDD), U10.26 (RUN), U10.30 (IOVDD), U10.38 (IOVDD), U10.44 (ADC_AVDD), U10.45 (IOVDD), U10.49 (VREG_VIN), U10.53 (USB_OTP_VDD), U10.54 (QSPI_IOVDD); no longer R15.2, R9.1
- net +5V: now also R51.1
- net +BATT: now also R1.2; no longer R1.1
- net 10V_ENABLE: now also U10.41 (GPIO27_ADC1)
- net ADC_VBAT: now also R1.1, U10.43 (GPIO29_ADC3); no longer R1.2
- net BEEPER: now also R23.2, Q5.1 (G), U10.28 (GPIO17)
- net BUZZER-: now also Q5.3 (D)
- net D+: now also R37.2
- net D-: now also R24.1
- net ESC_CURRENT: now also R9.1; no longer R6.2
- net FLASH_CS: now also U10.33 (GPIO21)
- net GND: now also C22.2, C37.2, C44.2, C45.2, C46.2, Q5.2 (S), Q6.2 (S), U10.47 (VREG_PGND), U10.61 (EP), U11.1; no longer C22.1
- net GYRO_CS: now also U10.17 (GPIO13); no longer R15.1
- net GYRO_INT: now also U10.13 (GPIO9)
- net LED0: now also R52.1, U10.40 (GPIO26_ADC0)
- net LED_STRIP: now also Q6.3 (D), R51.2
- net LED_STRIP_L: now also Q6.1 (G), U10.12 (GPIO8)
- net MOTOR1: now also U10.37 (GPIO25)
- net MOTOR2: now also U10.36 (GPIO24)
- net MOTOR3: now also U10.35 (GPIO23)
- net MOTOR4: now also U10.34 (GPIO22)
- net OSD_EN: now also U10.19 (GPIO15)
- net OSD_SYNC: now also U10.27 (GPIO16)
- net OSD_W: now also U10.18 (GPIO14)
- net PIOUART0_RX: now also U10.5 (GPIO3)
- net PIOUART0_TX: now also U10.4 (GPIO2)
- net SPI0.MISO: now also U10.32 (GPIO20)
- net SPI0.MOSI: now also U10.31 (GPIO19)
- net SPI0.SCK: now also U10.29 (GPIO18)
- net SPI1.MISO: now also U10.16 (GPIO12)
- net SPI1.MOSI: now also U10.15 (GPIO11)
- net SPI1.SCK: now also U10.14 (GPIO10)
- net UART0_RX: now also U10.3 (GPIO1)
- net UART0_TX: now also U10.2 (GPIO0)
- net UART1_RX: now also U10.10 (GPIO7)
- net UART1_TX: now also U10.9 (GPIO6)
- net XIN: now also U10.21 (XIN)
- net XOUT: now also U10.22 (XOUT)
- net ESC_CURR: now reaches R9.2
- net ESC_CURR: now also C22.1, U10.42 (GPIO28_ADC2)
- net at D2.2 (A): now also R53.2
- net RSSI renamed I2C0.SDA
- net I2C0.SDA: now also U10.7 (GPIO4)
- new net: R38.1, U11.2
- new net: R38.2, U10.60 (QSPI_SS)
- new net: R24.2, U10.51 (USB_DM)
- new net: C44.1, R15.2, U10.46 (VREG_AVDD)
- new net: R52.2, R53.1
- new net: L4.2, U10.48 (VREG_LX)
- new net: R37.1, U10.52 (USB_DP)
- new net I2C0.SCL: R6.2, U10.8 (GPIO5)
- no-connect marks 19 -> 9
Other:
- note added: "RP2350 1.1V DC-DC SMPS Follow datasheet guidance on component placement"
- note added: "RP2354A: Smaller variant with integrated flash (2MB)"
- note added: "USB port"
- note added: "decoupling caps, place close to IC, one is enough when 2 pins are next to each other"
- note added: "gyro SPI"
- note added: "i2c for external sensors"
- note added: "vbat sense. 1/11 scale"
- note removed: "1.1V SMPS by RP datasheet inductor polarity important"
- note removed: "RC lowpass filters on ADC and VREG like Pico datasheet"
- note removed: "RP2350 1.8V DC-DC SMPS Follow datasheet guidance on component placement"
- note removed: "RP2354B: Larger variant with integrated flash (2MB) and more GPIO"
- note removed: "USB port with ESD protection"
- note removed: "decoupling caps, place close to IC"
- note removed: "for external (extra)"
- note removed: "gyro SPI line, seperate from blackbox"
- note removed: "i2c for barometer and external sensors possibly"
- note removed: "vbat sense. 1/10 scale"
- moved on the sheet: C1, C10, C11, C12, C13, C3, C4, C5, C6, C7, C8, C9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
