File: hardware/rp2350a.kicad_sch (KiCad schematic)
At the start: 41 parts, among them Q5 AP1606, Q6 AP1606, U10 RP2354A, U11 TS2306A 240GF MSM 9_C2976675, X1 XTM25012000JT00351001

Commit message: docs(schematic): add design annotations to all sheets
Port on-canvas engineering comments from OpenFC-Lite (RP2354B), adapted to the
Mini layout. +41 text items across root, rp2350a, power, imu, osd, blackbox,
pads. Annotation/text only — no net or connectivity changes. Mirrors
hardware/DESIGN_NOTES.md.

Co-Authored-By: Claude Opus 4.8 (1M context) <noreply@anthropic.com>
Other:
- note added: "06/06/2026"
- note added: "2"
- note added: "RP2350 Pin mapping and universal peripherals"

Commit message: chore(bom): consolidate LCSC Part -> LCSC field across schematic, library, footprints, project
Single canonical LCSC field (was split LCSC / LCSC Part). Every part resolves to one LCSC code; netlist verified, no duplicates. Includes Rev2 re-annotation resync re-save.

Co-Authored-By: Claude Opus 4.8 (1M context) <noreply@anthropic.com>
Parts:
- L4: LCSC (none) -> C42411119; LCSC Part C42411119 -> (none)
- Q5, Q6: LCSC (none) -> C2849580; LCSC Part C2849580 -> (none)
- U10: LCSC (none) -> C41378174; LCSC Part C41378174 -> (none)
- U11: LCSC (none) -> C2976675; LCSC Part C2976675 -> (none)
- USB1: LCSC (none) -> C5187472; LCSC Part C5187472 -> (none)
- X1: LCSC (none) -> C37635340; LCSC Part C37635340 -> (none)
Changed lines of the file:
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@@
 			)
 		)
-		(property "LCSC Part" "C2976675"
+		(property "LCSC" "C2976675"
 			(at 247.65 217.17 0)
 			(hide yes)
@@
 			)
 		)
-		(property "LCSC Part" "C5187472"
+		(property "LCSC" "C5187472"
 			(at 110.49 265.43 0)
 			(hide yes)
@@
 			)
 		)
-		(property "LCSC Part" "C42411119"
+		(property "LCSC" "C42411119"
 			(at 257.81 245.11 0)
 			(hide yes)
@@
 			)
 		)
-		(property "LCSC Part" "C2849580"
+		(property "LCSC" "C2849580"
 			(at 429.26 208.28 0)
 			(hide yes)
@@
 			)
 		)
-		(property "LCSC Part" "C41378174"
+		(property "LCSC" "C41378174"
 			(at 295.91 290.83 0)
 			(hide yes)
@@
 			)
 		)
-		(property "LCSC Part" "C37635340"
+		(property "LCSC" "C37635340"
 			(at 140.97 256.54 0)
 			(hide yes)
@@
 			)
 		)
-		(property "LCSC Part" "C2849580"
+		(property "LCSC" "C2849580"
 			(at 422.91 148.59 0)
 			(hide yes)

Commit message: schematics: complete Manufacturer/MPN coverage, trim stray whitespace
22 field fixes across blackbox, osd, power, rp2350a: Manufacturer backfilled
from the LCSC catalogue, trailing space trimmed from four XL-1005UGC MPNs.
pads.kicad_sch (uncommitted WIP) untouched. Part of the fab-agnostic BOM
standardisation for quoting outside JLCPCB.

kicad-skip reflowed the touched files; structural diff shows only property
changes, ERC identical (163 violations before and after).

Co-Authored-By: Claude Fable 5 <noreply@anthropic.com>
Parts:
- R51: MPN (none) -> RTT012401FTH; Manufacturer (none) -> RALEC
