File: hardware/blackbox.kicad_sch (KiCad schematic)
At the start: 3 parts

Commit message: switch spi
Connections:
- net SPI1.MISO renamed SPI0.MISO
- net SPI1.MOSI renamed SPI0.MOSI
- net SPI1.SCK renamed SPI0.SCK
Changed lines of the file:
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@@
 	)
 	(bus_entry
-		(at 142.24 67.31)
+		(at 129.54 35.56)
 		(size 2.54 -2.54)
 		(stroke
@@
 	)
 	(bus_entry
-		(at 142.24 64.77)
+		(at 129.54 40.64)
 		(size 2.54 -2.54)
 		(stroke
@@
 	)
 	(bus_entry
-		(at 142.24 69.85)
+		(at 129.54 38.1)
 		(size 2.54 -2.54)
 		(stroke
@@
 	(bus
 		(pts
-			(xy 144.78 62.23) (xy 144.78 64.77)
-		)
-		(stroke
-			(width 0)
-			(type default)
-		)
-	)
-	(wire
-		(pts
-			(xy 128.27 69.85) (xy 142.24 69.85)
+			(xy 132.08 35.56) (xy 132.08 33.02)
+		)
+		(stroke
+			(width 0)
+			(type default)
+		)
+	)
+	(bus
+		(pts
+			(xy 132.08 33.02) (xy 153.67 33.02)
 		)
 		(stroke
@@
 		)
 	)
+	(wire
+		(pts
+			(xy 93.98 40.64) (xy 129.54 40.64)
+		)
+		(stroke
+			(width 0)
+			(type default)
+		)
+	)
 	(bus
 		(pts
-			(xy 144.78 64.77) (xy 144.78 67.31)
-		)
-		(stroke
-			(width 0)
-			(type default)
-		)
-	)
-	(wire
-		(pts
-			(xy 128.27 64.77) (xy 142.24 64.77)
+			(xy 132.08 38.1) (xy 132.08 35.56)
 		)
 		(stroke
@@
 	(wire
 		(pts
-			(xy 128.27 67.31) (xy 142.24 67.31)
-		)
-		(stroke
-			(width 0)
-			(type default)
-		)
-	)
-	(wire
-		(pts
 			(xy 59.69 50.8) (xy 58.42 50.8)
 		)
@@
 		)
 	)
-	(bus
-		(pts
-			(xy 152.4 62.23) (xy 144.78 62.23)
+	(wire
+		(pts
+			(xy 93.98 35.56) (xy 129.54 35.56)
+		)
+		(stroke
+			(width 0)
+			(type default)
+		)
+	)
+	(wire
+		(pts
+			(xy 93.98 38.1) (xy 129.54 38.1)
 		)
 		(stroke
@@
 		)
 	)
-	(label "SPI1.SCK"
+	(label "SPI0.MISO"
+		(at 96.52 35.56 0)
+		(effects
+			(font
+				(size 1.27 1.27)
+			)
+			(justify left bottom)
+		)
+	)
+	(label "SPI0.MOSI"
+		(at 96.52 38.1 0)
+		(effects
+			(font
+				(size 1.27 1.27)
+			)
+			(justify left bottom)
+		)
+	)
+	(label "SPI0.SCK"
 		(at 58.42 72.39 180)
 		(effects
@@
 		)
 	)
-	(label "SPI1.MISO"
-		(at 128.27 69.85 0)
-		(effects
-			(font
-				(size 1.27 1.27)
-			)
-			(justify left bottom)
-		)
-	)
-	(label "SPI1.MISO"
+	(label "SPI0.SCK"
+		(at 96.52 40.64 0)
+		(effects
+			(font
+				(size 1.27 1.27)
+			)
+			(justify left bottom)
+		)
+	)
+	(label "SPI0.MISO"
 		(at 86.36 72.39 0)
 		(effects
@@
 		)
 	)
-	(label "SPI1.MOSI"
-		(at 128.27 67.31 0)
-		(effects
-			(font
-				(size 1.27 1.27)
-			)
-			(justify left bottom)
-		)
-	)
-	(label "SPI1.SCK"
-		(at 128.27 64.77 0)
-		(effects
-			(font
-				(size 1.27 1.27)
-			)
-			(justify left bottom)
-		)
-	)
-	(label "SPI1.MOSI"
+	(label "SPI0.MOSI"
 		(at 58.42 69.85 180)
 		(effects
@@
 		)
 	)
-	(hierarchical_label "SPI1{SCK,MOSI,MISO}"
+	(hierarchical_label "SPI0{SCK,MOSI,MISO}"
 		(shape bidirectional)
-		(at 152.4 62.23 0)
-		(effects
-			(font
+		(at 153.67 33.02 0)
+		(effects
+			(font
