File: hardware/imu.kicad_sch (KiCad schematic)
At the start: 3 parts, among them U9 LSM6DSV16XTR

Commit message: Rev 2 (RP2354A): finalize design, update docs, clean repo (#5)
* docs(readme): add analog OSD BOM to Rev 2 change list

Document OSD debugging findings and component changes as a new
Analog OSD section in the Rev 2 Change List:
- HW-12: U19 op-amp TLV9061IDPWR -> COS8051SOT (175MHz video-grade RRIO)
- HW-13: output front-end add AC-couple + DC-restore, power U19 from +5V
- HW-14: U20 comparator TLV3201AIDBVR -> TLV7031DPWR (push-pull, X2SON, ~75% smaller)
- HW-15: add OSD_EN select pull-down (datasheet-required, defaults to pass-through)
- U18 / D9 verified correct, no change; OSD GPIO mapping noted (PA4/5/6)

Also fix HW-11 beeper GPIO: GPIO6 -> GPIO7 (GPIO6 is OSD_SYNC per netlist).

Co-Authored-By: Claude Opus 4.8 (1M context) <noreply@anthropic.com>

* many tiny improvements

- I/O correctness
- SPI0/SPI1/I2C0 bus corrections
- decoupling of DVDD
- ADC_AVDD as per RPi documents
- removal of SBUS
- connect ESC serial
- remove RUN RC-circuit as per RPi documentation
- some more cleanup for readability
- gyro CLKIN decision
- I2C 4.7k pullup

* RP2354A

* piu1

* switch spi

* Update OpenFC.kicad_pcb

* routex2

* some minor tweaks

- remove some unnecessary resistors
- slightly higher 10V rail to account for voltage drop
- some cleanup
- simpler PG 1.8V circuit

* Update imu.kicad_sch

* LED resistors

Also reduced the amount of different resistors for cheaper assembly

* Delete leds.kicad_sch

* remove some unneeded decoupling caps from RP2350

* update MOSFET part numbers

* OSD

* ROUTE

* clean libs

* details

* led names

* Clean routing

* docs: rewrite README + CLAUDE.md for finalized Rev 2 (RP2354A)

Rev 2 is a substantial redesign that the docs no longer matched. Updated
both to the actual schematic, verified from the current netlist:

- MCU: RP2354B (QFN-80, GPIO0-47) -> RP2354A (QFN-60, GPIO0-29). Full GPIO
  map re-derived from the netlist + QFN-60 pinout; all 30 GPIO documented.
- IMU moved to SPI1, microSD to SPI0; ref designators re-annotated
  (op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
Parts:
- added R49: 10k, Resistor_SMD:R_0201_0603Metric, symbol Device:R
Connections:
- net +3.3V: now also R49.2
- net GYRO_CS renamed CS
- net CS: now also R49.1
- net SPI0.CLKIN renamed CLKIN
- net SPI0.MISO renamed SPI1.MISO
- net SPI0.MOSI renamed SPI1.MOSI
- net SPI0.SCK renamed SPI1.SCK

Commit message: docs(schematic): add design annotations to all sheets
Port on-canvas engineering comments from OpenFC-Lite (RP2354B), adapted to the
Mini layout. +41 text items across root, rp2350a, power, imu, osd, blackbox,
pads. Annotation/text only — no net or connectivity changes. Mirrors
hardware/DESIGN_NOTES.md.

Co-Authored-By: Claude Opus 4.8 (1M context) <noreply@anthropic.com>
Other:
- note added: "06/06/2026"
- note added: "2"
- note added: "IMU SPI wiring and local decoupling"
- note added: "Universal IMU wiring and LGA footprint (BMI270, LSM6, TDK..)"

Commit message: chore(bom): consolidate LCSC Part -> LCSC field across schematic, library, footprints, project
Single canonical LCSC field (was split LCSC / LCSC Part). Every part resolves to one LCSC code; netlist verified, no duplicates. Includes Rev2 re-annotation resync re-save.

Co-Authored-By: Claude Opus 4.8 (1M context) <noreply@anthropic.com>
Parts:
- U9: LCSC (none) -> C5267406; LCSC Part C5267406 -> (none)
Changed lines of the file:
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@@
 			)
 		)
-		(property "LCSC Part" "C5267406"
+		(property "LCSC" "C5267406"
 			(at 72.39 87.63 0)
 			(hide yes)

Commit message: Swap 1.8V LDO and IMU, fix BOM/CPL export hygiene
Part changes, both schematic and PCB:
- U6 NCV8187AMT180TAG (stock 0 at JLC) replaced by U12 LP5912-1.8DRVR
  (C2876234). Same WSON-6 2x2 land pattern as the LP5912-3.3 at U7, so no
  layout change. PG is retained. PSRR at the 1 mA gyro load is ~85 dB to
  1 kHz and ~70 dB at 10 kHz per datasheet Figure 23.
- PG indicator rewired: pull-up from +5V to PG, LED from PG to GND, so the
  LED lights when the rail is good instead of when it has failed.
- U9 LSM6DSV16XTR replaced by BMI270 (C2836813). Bosch Table 22 matches the
  existing LGA-14 symbol pin for pin, so no rewire and no CPL rotation change.
- C33, C34 22uF 0402 moved from C105226 to C415703.

Export fixes:
- U12 carried its part number in a field named "LCSC Part" rather than
  "LCSC", so it exported with no part number and would have been quoted
  unsourced. Renamed.
- The 34 solder pad and testpoint footprints now carry exclude_from_bom
  plus exclude_from_pos_files instead of relying on the dnp flag. They stay
  on the board as copper but no longer need --exclude-dnp at export time.

BOM and CPL now agree at 101 placements with no blank part numbers, exported
without any dnp flag. ERC is unchanged against HEAD (170 vs 171 violations,
all pre-existing).

Co-Authored-By: Claude Fable 5 <noreply@anthropic.com>
Parts:
- U9: value LSM6DSV16XTR -> BMI270; LCSC C5267406 -> C2836813; MPN LSM6DSV16XTR -> BMI270; Manufacturer STMicroelectronics -> Bosch
Changed lines of the file:
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@@
 			)
 		)
-		(property "Value" "LSM6DSV16XTR"
+		(property "Value" "BMI270"
 			(at 60.96 70.866 0)
 			(show_name no)
@@
 			)
 		)
-		(property "LCSC" "C5267406"
+		(property "LCSC" "C2836813"
 			(at 72.39 87.63 0)
 			(hide yes)
@@
 			)
 		)
-		(property "MPN" "LSM6DSV16XTR"
+		(property "MPN" "BMI270"
 			(at 0 0 0)
 			(hide yes)
@@
 			)
 		)
-		(property "Manufacturer" "STMicroelectronics"
+		(property "Manufacturer" "Bosch"
 			(at 0 0 0)
 			(hide yes)
