File: hardware/OpenFC.kicad_pcb (KiCad board)
At the start: 6 copper layers, 37.5 x 37.5 mm, 164 parts, among them J1 5V, J10 5V, J11 5V, J12 5V, J13 5V, J14 5V, J15 5V, J18 5V, J2 5V, J21 5V, J22 5V, J25 5V, J26 5V, J27 5V, J28 5V, J29 5V, J30 5V, J31 5V, J32 5V, J33 5V, J34 5V, J35 5V, J36 5V, J37 5V, J38 5V, J39 5V, J4 5V, J40 5V, J41 5V, J42 5V, J43 5V, J44 5V, J45 5V, J46 5V, J47 5V, J48 5V, J49 5V, J5 5V, J50 5V, J52 5V, J53 5V, J54 5V, J7 5V, J8 5V, P1 SM08B-SRSS-TB(LF)(SN), Q1 DMN1150UFB-7B, Q2 DMN1150UFB-7B, Q3 DMN1150UFB-7B, Q4 DMN1150UFB-7B, U1 TS2306A 240GF MSM 9_C2976675, U18 SN74LVC1G3157DTBR, U19 TLV9061IDPWR, U2 RP2354B_C39843328, U20 TLV3201AIDBVR, U3 LMR51420YFDDCR, U4 LMR51420YFDDCR, U5 TPS2116DRLR, U6 NCV8187AMT180TAG, U7 LP5912-3.3DRVR, U8 SM06B-SRSS-TB(LF)(SN), U9 LSM6DSV16XTR, X1 XTM25012000JT00351001

Commit message: switch spi
Parts:
- removed C14, C15, C16, C2: 100n, Capacitor_SMD:C_0201_0603Metric
- removed C18, C20, C23: 4.7uF, Capacitor_SMD:C_0402_1005Metric
- removed D1: USBLC6-2P6, Package_TO_SOT_SMD:SOT-666
- removed D10: LED_1_Green, LED_SMD:LED_0201_0603Metric
- removed J1, J11, J13, J2, J36, J38, J47, J50, J52, J53, J54: 5V, lib:small_pad
- removed L1: AOTA-B201610S3R3-101-T, lib:IND-SMD_L2.0-W1.6_AOTA-B201610S3R3-101-T
- removed Q1: DMN1150UFB-7B, lib:DFN-3L_L1.0-W0.6-P0.65-BR
- removed R10, R11: 10k, Resistor_SMD:R_0201_0603Metric
- removed R12, R13, R14: 30R, Resistor_SMD:R_0201_0603Metric
- removed R17, R18: 2.2k, Resistor_SMD:R_0201_0603Metric
- removed R6, R7, R8: 1k, Resistor_SMD:R_0201_0603Metric
- removed U1: TS2306A 240GF MSM 9_C2976675, lib:SW-SMD_4P-L3.0-W2.0-P0.85-LS3.5
- removed U2: RP2354B_C39843328, lib:QFN-80_L10.0-W10.0-P0.40-TL-EP3.4
- added C37: 4.7uF, Capacitor_SMD:C_0402_1005Metric, F.Cu at (49.1, 52.9)
- added C44: 4.7uF, Capacitor_SMD:C_0402_1005Metric, F.Cu at (49.1, 54.9)
- added C45: 4.7uF, Capacitor_SMD:C_0402_1005Metric, F.Cu at (49.1, 56.8)
- added C46: 4.7uF, Capacitor_SMD:C_0402_1005Metric, F.Cu at (49.1, 58.8)
- added D8: LED_1_Green, LED_SMD:LED_0402_1005Metric, B.Cu at (177.4, 76.8)
- added L4: AOTA-B201610S3R3-101-T, lib:IND-SMD_L2.0-W1.6_AOTA-B201610S3R3-101-T, F.Cu at (47.6, 66.0)
- added R37: 30R, Resistor_SMD:R_0201_0603Metric, F.Cu at (44.4, 63.6)
- added R38: 10k, Resistor_SMD:R_0201_0603Metric, F.Cu at (44.4, 65.3)
- added R49: 10k, Resistor_SMD:R_0201_0603Metric, F.Cu at (171.1, 86.6)
- added U10: RP2354A, lib:QFN-60_L7.0-W7.0-P0.40-TL-EP3.4, F.Cu at (108.5, 63.3)
- added U11: TS2306A 240GF MSM 9_C2976675, lib:SW-SMD_4P-L3.0-W2.0-P0.85-LS3.5, F.Cu at (48.0, 62.6)
- C21: value 4.7uF -> 100n; footprint Capacitor_SMD:C_0402_1005Metric -> Capacitor_SMD:C_0201_0603Metric; moved to F.Cu
- C22, C35, C36, C43, J10, J4, J7, U9: moved to F.Cu
- D2: value LED_1_Green -> LED_1_Blue; footprint LED_SMD:LED_0201_0603Metric -> LED_SMD:LED_0402_1005Metric
- D4, D5: footprint LED_SMD:LED_0201_0603Metric -> LED_SMD:LED_0402_1005Metric; moved to B.Cu
- D7: footprint LED_SMD:LED_0201_0603Metric -> LED_SMD:LED_0402_1005Metric
- R15, R24: value 10k -> 30R; moved to F.Cu
- R19: value 1k -> 4.7k; moved to F.Cu
- R21: value 100k -> 4.7k; moved to F.Cu
- R30: value 6.8k -> 6.49k
- R9: value 200R -> 1k; moved to F.Cu
- U3, U4: value LMR51420YFDDCR -> TI LMR51430YFDDCR
- moved R15 116.4 mm to (41.9, 61.8), turned to 0 degrees
- moved C22 111.8 mm to (39.5, 63.6), turned to 0 degrees
- moved R21 111.4 mm to (41.9, 65.3), turned to 0 degrees
- moved C21 111.0 mm to (39.5, 61.8), turned to 0 degrees
- moved R9 111.0 mm to (39.5, 65.3), turned to 0 degrees
- moved R19 110.9 mm to (41.9, 63.6), turned to 0 degrees
- moved R24 109.9 mm to (44.4, 61.8), turned to 0 degrees
- moved C10 71.7 mm to (87.6, 56.5)
- moved C17 71.7 mm to (80.1, 66.3)
- moved C6 71.7 mm to (87.6, 57.8)
- moved C1 71.7 mm to (83.8, 58.7)
- moved C11 71.7 mm to (87.0, 58.8)
- moved C12 71.7 mm to (81.3, 59.4)
- moved C13 71.7 mm to (81.2, 62.3)
- moved C19 71.7 mm to (85.6, 58.8)
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Connections:
- net /LED renamed /PADS/LED_STRIP
- net /PADS/DIGITAL_RX renamed /PADS/UART0_RX
- net /PADS/DIGITAL_TX renamed /PADS/UART0_TX
- C21 pad 1: Net-(U2-ADC_AVDD) -> +3.3V
- C22 pad 1: GND -> /RP2350A/ESC_CURR
- C22 pad 2: Net-(U2-RUN) -> GND
- J12 pad 1: /UART1_TX -> /PADS/UART1_TX
- J15 pad 1: /I2C_SCL -> /PADS/I2C0.SCL
- J18 pad 1: /I2C_SDA -> /PADS/I2C0.SDA
- J44 pad 1: /PADS/PIOUART0_RX -> /PADS/PU0RX
- J8 pad 1: /UART1_RX -> /PADS/U1RX
- P1 pad 4: unconnected-(P1-Pad4) -> /PADS/PU0RX
- R1 pad 1: +BATT -> /RP2350A/ADC_VBAT
- R1 pad 2: /RP2350A/ADC_VBAT -> +BATT
- R15 pad 1: /IMU/GYRO_CS -> +3.3V
- R15 pad 2: +3.3V -> Net-(U10-VREG_AVDD)
- R19 pad 1: Net-(Q1-G) -> /PADS/I2C0.SCL
- R19 pad 2: /PADS/SBUS -> +3.3V
- R21 pad 1: GND -> /PADS/I2C0.SDA
- R21 pad 2: Net-(Q1-G) -> +3.3V
- R24 pad 1: /RP2350A/SBUS_INVERT -> /RP2350A/D-
- R24 pad 2: +3.3V -> Net-(U10-USB_DM)
- R9 pad 1: +3.3V -> /PADS/CURRENT
- R9 pad 2: Net-(U2-ADC_AVDD) -> /RP2350A/ESC_CURR
- U8 pad 6: /PADS/SBUS -> /PADS/U1RX
- U9 pad 12: /IMU/GYRO_CS -> /IMU/CS
- U9 pad 9: /IMU/SPI0.CLKIN -> /IMU/CLKIN
- USB1 pad A6: /RP2350A/D+_C -> /RP2350A/D+
- USB1 pad A7: /RP2350A/D-_C -> /RP2350A/D-
- USB1 pad B6: /RP2350A/D+_C -> /RP2350A/D+
- USB1 pad B7: /RP2350A/D-_C -> /RP2350A/D-
Routing:
- net GND: track 106.8 -> 7.51 mm, vias 61 -> 0
- net +3.3V: track 87.7 -> 0.00 mm, vias 31 -> 0
- net +BATT: track 70.5 -> 4.75 mm, vias 9 -> 0
- net +10V: track 56.2 -> 0.00 mm, vias 5 -> 0
- net +1.1V: track 31.0 -> 0.00 mm, vias 5 -> 0
- net +5V: track 29.9 -> 0.00 mm, vias 21 -> 0
- net /BLACKBOX/SPI1.MISO: track 21.6 -> 0.00 mm, vias 2 -> 0
- net /POWER/10V_ENABLE: track 19.9 -> 0.00 mm, vias 2 -> 0
- net /BLACKBOX/FLASH_CS: track 18.3 -> 0.00 mm, vias 2 -> 0
- net /BLACKBOX/SPI1.SCK: track 16.9 -> 0.00 mm, vias 2 -> 0
- net /RP2350A/LED0: track 16.3 -> 0.00 mm, vias 2 -> 0
- net Net-(D8-K): track 16.0 -> 0.00 mm, vias 2 -> 0
- net /BLACKBOX/SPI1.MOSI: track 15.9 -> 0.00 mm, vias 2 -> 0
- net /PADS/RSSI: track 15.6 -> 0.00 mm, vias 2 -> 0
- net /OSD/VIDEO_IN: track 14.5 -> 0.00 mm, vias 1 -> 0
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- removed copper zone on In2.Cu, net GND
Other:
- board size 37.5 x 37.5 mm -> 27.6 x 27.6 mm
- board text removed: "10V"
- board text removed: "ADC"
- board text removed: "RSSI"
- board text removed: "RX4"
- board text removed: "SBUS"
- board text removed: "TX4"

Commit message: Update OpenFC.kicad_pcb
Parts:
- removed R26: 200R, Resistor_SMD:R_0201_0603Metric
- C10, C31, C33, C6, D8, Q4, R16, R35, R40, R5, U6, X1: moved to F.Cu
- C21, C22, C37, C43, C44, C45, C46, D7, L4, R15, R24, R37, R9, U10: moved to B.Cu
- moved C21 122.4 mm to (159.0, 87.9)
- moved C37 112.7 mm to (154.9, 91.9)
- moved C22 112.0 mm to (149.5, 84.4), turned to 180 degrees
- moved R9 111.6 mm to (149.5, 83.7)
- moved R37 111.5 mm to (154.4, 81.8), turned to 90 degrees
- moved R24 111.1 mm to (153.7, 81.8), turned to -90 degrees
- moved R15 110.6 mm to (150.6, 82.6), turned to 90 degrees
- moved C45 106.2 mm to (152.2, 82.3), turned to 180 degrees
- moved C46 105.5 mm to (152.2, 81.4), turned to 180 degrees
- moved L4 105.4 mm to (152.1, 80.0), turned to 180 degrees
- moved C44 104.7 mm to (150.4, 81.4), turned to 180 degrees
- moved R25 77.8 mm to (159.0, 90.2), turned to 0 degrees
- moved C17 77.6 mm to (153.4, 91.6), turned to -90 degrees
- moved R5 77.3 mm to (154.3, 90.5)
- moved R22 77.0 mm to (159.0, 88.6), turned to 180 degrees
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Connections:
- Card1 pad 3: /BLACKBOX/SPI1.MOSI -> /BLACKBOX/SPI0.MOSI
- Card1 pad 5: /BLACKBOX/SPI1.SCK -> /BLACKBOX/SPI0.SCK
- Card1 pad 7: /BLACKBOX/SPI1.MISO -> /BLACKBOX/SPI0.MISO
- Q3 pad 3: Net-(Q3-D) -> /PADS/LED_STRIP
- R25 pad 2: Net-(Q3-D) -> /PADS/LED_STRIP
- U10 pad 10: /RP2350A/LED_STRIP_L -> /PADS/U1RX
- U10 pad 12: /PADS/UART1_TX -> /RP2350A/LED_STRIP_L
- U10 pad 13: /PADS/U1RX -> /IMU/GYRO_INT
- U10 pad 14: /BLACKBOX/SPI1.SCK -> /IMU/SPI1.SCK
- U10 pad 15: /BLACKBOX/SPI1.MOSI -> /IMU/SPI1.MOSI
- U10 pad 16: /BLACKBOX/SPI1.MISO -> /IMU/SPI1.MISO
- U10 pad 17: /BLACKBOX/FLASH_CS -> /IMU/CS
- U10 pad 28: /IMU/GYRO_INT -> /RP2350A/BEEPER
- U10 pad 29: /IMU/SPI0.SCK -> /BLACKBOX/SPI0.SCK
- U10 pad 31: /IMU/SPI0.MOSI -> /BLACKBOX/SPI0.MOSI
- U10 pad 32: /IMU/SPI0.MISO -> /BLACKBOX/SPI0.MISO
- U10 pad 33: /IMU/CS -> /BLACKBOX/FLASH_CS
- U10 pad 7: /PADS/I2C0.SCL -> /PADS/I2C0.SDA
- U10 pad 8: /PADS/I2C0.SDA -> /PADS/I2C0.SCL
- U10 pad 9: /RP2350A/BEEPER -> /PADS/UART1_TX
- U9 pad 1: /IMU/SPI0.MISO -> /IMU/SPI1.MISO
- U9 pad 13: /IMU/SPI0.SCK -> /IMU/SPI1.SCK
- U9 pad 14: /IMU/SPI0.MOSI -> /IMU/SPI1.MOSI
Routing:
- net +3.3V: track 0.00 -> 15.1 mm
- net GND: track 7.51 -> 21.6 mm, vias 0 -> 1
- net +1.1V: track 0.00 -> 7.86 mm
- net +5V_BUCK: track 2.34 -> 10.1 mm
- net /PADS/M4: track 0.00 -> 7.23 mm, vias 0 -> 1
- net /PADS/M3: track 0.00 -> 6.56 mm, vias 0 -> 1
- net +5V: track 0.00 -> 6.32 mm
- net /PADS/M2: track 0.00 -> 5.79 mm, vias 0 -> 1
- net +BATT: track 4.75 -> 0.00 mm
- net /PADS/M1: track 0.00 -> 3.86 mm, vias 0 -> 1
- net Net-(U10-VREG_LX): track 0.00 -> 3.69 mm
- net Net-(C10-Pad2): track 0.00 -> 3.60 mm
- net /RP2350A/ADC_VBAT: track 0.00 -> 2.91 mm
- net Net-(U10-VREG_AVDD): track 0.00 -> 2.37 mm
- net /RP2350A/ESC_CURR: track 0.00 -> 1.95 mm
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Other:
- outline, holes or cut-outs redrawn
