File: hardware/OpenFC.kicad_pcb (KiCad board)
At the start: 6 copper layers, 27.6 x 27.6 mm, 140 parts, among them J10 5V, J12 5V, J14 5V, J15 5V, J18 5V, J21 5V, J22 5V, J25 5V, J26 5V, J27 5V, J28 5V, J29 5V, J30 5V, J31 5V, J32 5V, J33 5V, J34 5V, J35 5V, J37 5V, J39 5V, J4 5V, J40 5V, J41 5V, J42 5V, J43 5V, J44 5V, J45 5V, J46 5V, J48 5V, J49 5V, J5 5V, J7 5V, J8 5V, P1 SM08B-SRSS-TB(LF)(SN), Q2 DMN1150UFB-7B, Q3 DMN1150UFB-7B, Q4 DMN1150UFB-7B, U10 RP2354A, U11 TS2306A 240GF MSM 9_C2976675, U18 SN74LVC1G3157DTBR, U19 TLV9061IDPWR, U20 TLV3201AIDBVR, U3 TI LMR51430YFDDCR, U4 TI LMR51430YFDDCR, U5 TPS2116DRLR, U6 NCV8187AMT180TAG, U7 LP5912-3.3DRVR, U8 SM06B-SRSS-TB(LF)(SN), U9 LSM6DSV16XTR, X1 XTM25012000JT00351001

Commit message: ROUTE
Parts:
- removed C17, C19, C21: 100n, Capacitor_SMD:C_0201_0603Metric
- removed D6: RB161QS-40_C28646385, lib:SOD-882_L1.0-W0.6-RD
- removed J4, J7: 5V, lib:small_pad
- removed Q2, Q3, Q4: DMN1150UFB-7B, lib:DFN-3L_L1.0-W0.6-P0.65-BR
- removed R16: 30R, Resistor_SMD:R_0201_0603Metric
- removed R19, R21: 4.7k, Resistor_SMD:R_0201_0603Metric
- removed R20: 1k, Resistor_SMD:R_0201_0603Metric
- removed R22, R25: 2.2k, Resistor_SMD:R_0201_0603Metric
- removed R34: 200R, Resistor_SMD:R_0201_0603Metric
- removed R35: 10k, Resistor_SMD:R_0201_0603Metric
- removed U19: TLV9061IDPWR, lib:X2SON-4_L0.8-W0.8-P0.48-TL-DPW
- removed U20: TLV3201AIDBVR, lib:SOT-23-5_L3.0-W1.7-P0.95-LS2.8-BR
- added D10: RB161QS-40_C28646385, lib:SOD-882_L1.0-W0.6-RD, B.Cu at (147.6, 90.1)
- added J17: 5V, lib:small_pad, F.Cu at (140.9, 87.5)
- added J20: 5V, lib:small_pad, F.Cu at (140.9, 89.8)
- added J24: 5V, lib:small_pad, F.Cu at (140.9, 92.1)
- added Q5: AP1606, lib:DFN-3L_L1.0-W0.6-P0.65-BR, B.Cu at (158.9, 85.4)
- added Q6: AP1606, lib:DFN-3L_L1.0-W0.6-P0.65-BR, B.Cu at (153.2, 92.2)
- added R50: 2.4k, Resistor_SMD:R_0201_0603Metric, F.Cu at (146.4, 80.7)
- added R51: 2.4k, Resistor_SMD:R_0201_0603Metric, B.Cu at (152.6, 92.2)
- added R52: 75R, Resistor_SMD:R_0201_0603Metric, B.Cu at (157.4, 78.4)
- added R53: 75R, Resistor_SMD:R_0201_0603Metric, F.Cu at (158.5, 80.3)
- added R6: 5.1k, Resistor_SMD:R_0201_0603Metric, B.Cu at (150.7, 91.4)
- added R7: 5.1k, Resistor_SMD:R_0201_0603Metric, B.Cu at (150.7, 90.7)
- added U1: COS8051SOT, lib:SOT-23-5_L3.0-W1.7-P0.95-LS2.8-BR, B.Cu at (157.8, 92.0)
- added U2: TLV7031DPWR, lib:X2SON-4_L0.8-W0.8-P0.48-TL-A, B.Cu at (158.3, 89.2)
- C1, C12, C13, C22, C27, C4, C44, C45, C46, C9, D4, D5, D7, L4, R1, R15, R2, R24, R31, R32, R37, R4, R9, U10: moved to F.Cu
- C10, C6, R49, R5, X1: moved to B.Cu
- R33: value 470R -> 7.5k; moved to F.Cu
- R36: value 30R -> 510R; moved to F.Cu
- R40: value 200R -> 2.4k
- R46, R47: value 470R -> 510R
- moved R38 56.9 mm to (147.8, 90.9)
- moved R49 53.3 mm to (155.0, 93.4), turned to 180 degrees
- moved U11 51.9 mm to (145.8, 89.5), turned to -90 degrees
- moved J10 38.4 mm to (164.5, 80.8)
- moved J21 35.1 mm to (160.6, 82.0), turned to 0 degrees
- moved J25 34.4 mm to (160.6, 84.3), turned to 0 degrees
- moved R45 32.4 mm to (156.8, 85.9), turned to 90 degrees
- moved R41 32.1 mm to (157.5, 85.9), turned to 90 degrees
- moved C38 31.8 mm to (158.2, 85.9), turned to 90 degrees
- moved U18 30.2 mm to (157.1, 87.3), turned to 90 degrees
- moved R48 29.6 mm to (159.1, 94.4)
- moved C40 29.5 mm to (158.3, 87.5), turned to -90 degrees
- moved C39 29.1 mm to (157.1, 88.2), turned to 180 degrees
- moved C41 29.0 mm to (159.6, 92.1), turned to 180 degrees
- moved C42 28.6 mm to (158.5, 90.2)
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Connections:
- R23 pad 2: Net-(Q2-G) -> /RP2350A/BEEPER
- R40 pad 2: Net-(Q4-D) -> /POWER/1.8V_PG
- R46 pad 1: GND -> Net-(U1-IN-)
- R46 pad 2: Net-(U19-IN-) -> GND
- R47 pad 1: Net-(U19-IN-) -> Net-(U1-IN-)
- U10 pad 40: /RP2350A/ADC_VBAT -> /RP2350A/LED0
- U10 pad 41: /RP2350A/ESC_CURR -> /POWER/10V_ENABLE
- U10 pad 42: /POWER/10V_ENABLE -> /RP2350A/ESC_CURR
- U10 pad 43: /RP2350A/LED0 -> /RP2350A/ADC_VBAT
Routing:
- net GND: track 21.6 -> 82.4 mm, vias 1 -> 75
- net /PADS/LED_STRIP: track 0.83 -> 53.4 mm, vias 0 -> 3
- net +BATT: track 0.00 -> 38.6 mm, vias 0 -> 4
- net +10V: track 1.21 -> 33.1 mm, vias 0 -> 7
- net +5V: track 6.32 -> 38.1 mm, vias 0 -> 20
- net /PADS/PU0RX: track 0.00 -> 28.4 mm, vias 0 -> 3
- net +3.3V: track 15.1 -> 43.2 mm, vias 0 -> 16
- net /PADS/U1RX: track 0.02 -> 26.2 mm, vias 1 -> 3
- net +1.1V: track 7.86 -> 29.5 mm, vias 0 -> 5
- net /PADS/PIOUART0_TX: track 0.00 -> 20.3 mm, vias 0 -> 2
- net /PADS/UART0_RX: track 0.00 -> 16.5 mm, vias 0 -> 2
- net /PADS/I2C0.SCL: track 0.80 -> 16.3 mm, vias 1 -> 2
- net /PADS/I2C0.SDA: track 0.53 -> 15.1 mm, vias 1 -> 2
- net /PADS/UART1_TX: track 0.85 -> 14.6 mm, vias 1 -> 2
- net /PADS/UART0_TX: track 0.00 -> 13.6 mm, vias 0 -> 3
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- added copper zone on In3.Cu, net +3.3V
- added copper zone on In2.Cu, net GND
- removed copper zone on In2.Cu, net +3.3V
Other:
- board text added: "LITE"
- board text added: "RP0"
- board text added: "RX0"
- board text added: "TP0"
- board text added: "TX0"
- board text removed: "+5v"
- board text removed: "gnd"
- board text removed: "led"

Commit message: clean libs
Routing:
- net GND: track 82.4 -> 84.7 mm, vias 75 -> 78
Changed lines of the file:
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@@
 		(model "${KIPRJMOD}/lib.3dshapes/DFN-3L_L1.0-W0.6-H0.5-P0.65-BR.wrl"
 			(offset
-				(xyz 0.01 -0 -0)
+				(xyz 0.01 -0 0.5)
 			)
 			(scale
@@
 			)
 			(rotate
-				(xyz 0 0 0)
+				(xyz -0 -0 -0)
 			)
 		)
@@
 		(sheetname "/OSD/")
 		(sheetfile "osd.kicad_sch")
+		(units
+			(unit
+				(name "A")
+				(pins "3" "1" "5" "2" "4" "6")
+			)
+		)
 		(attr smd)
 		(duplicate_pad_numbers_are_jumpers no)
@@
 		(sheetname "/OSD/")
 		(sheetfile "osd.kicad_sch")
+		(units
+			(unit
+				(name "A")
+				(pins "3" "4" "2" "5" "1")
+			)
+		)
 		(attr smd)
 		(duplicate_pad_numbers_are_jumpers no)
@@
 	)
 	(via
+		(at 162.65 91.29)
+		(size 0.35)
+		(drill 0.2)
+		(layers "F.Cu" "B.Cu")
+		(net "GND")
+	)
+	(via
 		(at 141.04 93.93)
 		(size 0.35)
@@
 	)
 	(via
+		(at 162.57 81.0625)
+		(size 0.35)
+		(drill 0.2)
+		(layers "F.Cu" "B.Cu")
+		(net "GND")
+	)
+	(via
 		(at 147.28 82.8)
 		(size 0.35)
@@
 	)
 	(via
+		(at 162.02 81.07)
+		(size 0.35)
+		(drill 0.2)
+		(layers "F.Cu" "B.Cu")
+		(net "GND")
+	)
+	(via
 		(at 151.486264 92.995336)
 		(size 0.35)
@@
 	)
 	(segment
+		(start 162.75 91.39)
+		(end 162.65 91.29)
+		(width 0.1)
+		(layer "B.Cu")
+		(net "GND")
+	)
+	(segment
 		(start 141.13 93.93)
 		(end 141.545852 93.93)
@@
 	)
 	(segment
+		(start 162.57 81.0625)
+		(end 162.0275 81.0625)
+		(width 0.2)
+		(layer "B.Cu")
+		(net "GND")
+	)
+	(segment
 		(start 153.997106 92.455)
 		(end 153.47 91.927894)
@@
 	)
 	(segment
+		(start 162.75 91.9025)
+		(end 162.75 91.39)
+		(width 0.1)
+		(layer "B.Cu")
+		(net "GND")
+	)
+	(segment
 		(start 156.84 88.17)
 		(end 156.75 88.26)
@@
 	)
 	(segment
+		(start 163.5 81.0625)
+		(end 162.4175 81.0625)
+		(width 0.09)
+		(layer "B.Cu")
+		(net "GND")
+	)
+	(segment
 		(start 144.334898 81.5475)
 		(end 144.05 81.5475)
@@
 	)
 	(segment
+		(start 162.0275 81.0625)
+		(end 162.02 81.07)
+		(width 0.2)
+		(layer "B.Cu")
+		(net "GND")
+	)
+	(segment
 		(start 145.92 91.96)
 		(end 145.75 92.13)
@@
 	)
 	(segment
+		(start 158.474851 92.604851)
+		(end 159.067053 93.197053)
+		(width 0.3)
+		(layer "F.Cu")
+		(net "Net-(D7-A)")
+	)
+	(segment
 		(start 160.6 82.05)
 		(end 158.65 84)
@@
 	)
 	(segment
+		(start 146.271716 92.59)
+		(end 145.766585 93.095131)
+		(width 0.3)
+		(layer "F.Cu")
+		(net "Net-(D4-A)")
+	)
+	(segment
+		(start 146.43 92.59)
+		(end 146.271716 92.59)
+		(width 0.3)
+		(layer "F.Cu")
+		(net "Net-(D4-A)")
+	)
+	(segment
 		(start 154.81 79.85)
 		(end 154.45 80.21)
@@
 	)
 	(segment
+		(start 146.143726 80.433726)
+		(end 146.129583 80.433726)
+		(width 0.2)
+		(layer "F.Cu")
+		(net "Net-(D5-A)")
+	)
+	(segment
+		(start 146.129583 80.433726)
+		(end 145.59395 79.898093)
+		(width 0.2)
+		(layer "F.Cu")
+		(net "Net-(D5-A)")
+	)
+	(segment
 		(start 148.61 78.81)
 		(end 148.33 78.81)
@@
 	)
 	(segment
-		(start 148.18 92.08)
-		(end 148.18 94.34)
-		(width 0.2)
-		(layer "F.Cu")
-		(net "Net-(U3-SW)")
-	)
-	(segment
-		(start 148.18 94.34)
-		(end 147.64 94.88)
-		(width 0.2)
-		(layer "F.Cu")
-		(net "Net-(U3-SW)")
-	)
-	(via
-		(at 147.64 94.88)
-		(size 0.35)
-		(drill 0.2)
-		(layers "F.Cu" "B.Cu")
-		(net "Net-(U3-SW)")
-	)
-	(via
-		(at 148.18 92.08)
-		(size 0.35)
-		(drill 0.2)
-		(layers "F.Cu" "B.Cu")
-		(net "Net-(U3-SW)")
-	)
-	(segment
-		(start 147.6675 95.27)
-		(end 147.6675 94.9075)
-		(width 0.6)
-		(layer "B.Cu")
-		(net "Net-(U3-SW)")
-	)
-	(segment
-		(start 146.76 97.209976)
-		(end 146.76 97.66)
-		(width 0.6)
-		(layer "B.Cu")
-		(net "Net-(U3-SW)")
-	)
-	(segment
-		(start 148.214605 91.953687)
-		(end 148.214605 92.045395)
-		(width 0.2)
-		(layer "B.Cu")
-		(net "Net-(U3-SW)")
-	)
-	(segment
-		(start 147.6675 95.27)
-		(end 147.6675 96.302476)
-		(width 0.6)
-		(layer "B.Cu")
-		(net "Net-(U3-SW)")
-	)
-	(segment
-		(start 147.6675 94.9075)
-		(end 147.64 94.88)
-		(width 0.6)
-		(layer "B.Cu")
-		(net "Net-(U3-SW)")
-	)
-	(segment
-		(start 147.6675 96.302476)
-		(end 146.76 97.209976)
-		(width 0.6)
-		(layer "B.Cu")
-		(net "Net-(U3-SW)")
-	)
-	(segment
-		(start 148.214605 92.045395)
-		(end 148.18 92.08)
-		(width 0.2)
-		(layer "B.Cu")
-		(net "Net-(U3-SW)")
-	)
-	(segment
-		(start 148.854605 92.732895)
-		(end 148.6175 92.97)
-		(width 0.2)
-		(layer "B.Cu")
-		(net "Net-(U3-CB)")
-	)
-	(segment
-		(start 148.854605 91.953687)
-		(end 148.854605 92.732895)
-		(width 0.2)
-		(layer "B.Cu")
-		(net "Net-(U3-CB)")
-	)
-	(segment
 		(start 158.242356 80.549065)
 		(end 158.11 80.416709)
@@
 	)
 	(segment
-		(start 158.474851 92.604851)
-		(end 159.067053 93.197053)
-		(width 0.3)
-		(layer "F.Cu")
-		(net "Net-(D7-A)")
-	)
-	(segment
 		(start 159.403726 93.726274)
 		(end 160.033726 93.726274)
@@
 	)
 	(segment
-		(start 146.271716 92.59)
-		(end 145.766585 93.095131)
-		(width 0.3)
+		(start 148.18 92.08)
+		(end 148.18 94.34)
+		(width 0.2)
 		(layer "F.Cu")
-		(net "Net-(D4-A)")
+		(net "Net-(U3-SW)")
 	)
 	(segment
-		(start 146.43 92.59)
-		(end 146.271716 92.59)
-		(width 0.3)
+		(start 148.18 94.34)
+		(end 147.64 94.88)
+		(width 0.2)
 		(layer "F.Cu")
-		(net "Net-(D4-A)")
+		(net "Net-(U3-SW)")
+	)
+	(via
+		(at 147.64 94.88)
+		(size 0.35)
+		(drill 0.2)
+		(layers "F.Cu" "B.Cu")
+		(net "Net-(U3-SW)")
+	)
+	(via
+		(at 148.18 92.08)
+		(size 0.35)
+		(drill 0.2)
+		(layers "F.Cu" "B.Cu")
+		(net "Net-(U3-SW)")
+	)
+	(segment
+		(start 147.6675 95.27)
+		(end 147.6675 94.9075)
+		(width 0.6)
+		(layer "B.Cu")
+		(net "Net-(U3-SW)")
+	)
+	(segment
+		(start 146.76 97.209976)
+		(end 146.76 97.66)
+		(width 0.6)
+		(layer "B.Cu")
+		(net "Net-(U3-SW)")
+	)
+	(segment
+		(start 148.214605 91.953687)
+		(end 148.214605 92.045395)
+		(width 0.2)
+		(layer "B.Cu")
+		(net "Net-(U3-SW)")
+	)
+	(segment
+		(start 147.6675 95.27)
+		(end 147.6675 96.302476)
+		(width 0.6)
+		(layer "B.Cu")
+		(net "Net-(U3-SW)")
+	)
+	(segment
+		(start 147.6675 94.9075)
+		(end 147.64 94.88)
+		(width 0.6)
+		(layer "B.Cu")
+		(net "Net-(U3-SW)")
+	)
+	(segment
+		(start 147.6675 96.302476)
+		(end 146.76 97.209976)
+		(width 0.6)
+		(layer "B.Cu")
+		(net "Net-(U3-SW)")
+	)
+	(segment
+		(start 148.214605 92.045395)
+		(end 148.18 92.08)
+		(width 0.2)
+		(layer "B.Cu")
+		(net "Net-(U3-SW)")
 	)
 	(segment
@@
 	)
 	(segment
-		(start 146.143726 80.433726)
-		(end 146.129583 80.433726)
-		(width 0.2)
-		(layer "F.Cu")
-		(net "Net-(D5-A)")
-	)
-	(segment
-		(start 146.129583 80.433726)
-		(end 145.59395 79.898093)
-		(width 0.2)
-		(layer "F.Cu")
-		(net "Net-(D5-A)")
-	)
-	(segment
 		(start 159.600374 91.09)
 		(end 159.13 91.09)
@@
 	)
 	(segment
+		(start 148.854605 92.732895)
+		(end 148.6175 92.97)
+		(width 0.2)
+		(layer "B.Cu")
+		(net "Net-(U3-CB)")
+	)
+	(segment
+		(start 148.854605 91.953687)
+		(end 148.854605 92.732895)
+		(width 0.2)
+		(layer "B.Cu")
+		(net "Net-(U3-CB)")
+	)
+	(segment
 		(start 145.75 90.18)
 		(end 146.61 90.18)
@@
 		(layer "F.Cu")
 		(hatch none 0.1)
-		(priority 30004)
+		(priority 30007)
 		(attr
 			(teardrop
@@
 		(layer "F.Cu")
 		(hatch none 0.1)
-		(priority 30005)
+		(priority 30006)
 		(attr
 			(teardrop
@@
 		(layer "F.Cu")
 		(hatch none 0.1)
-		(priority 30007)
+		(priority 30004)
 		(attr
 			(teardrop
@@
 		(layer "F.Cu")
 		(hatch none 0.1)
-		(priority 30003)
+		(priority 30005)
 		(attr
 			(teardrop
@@
 		(layer "F.Cu")
 		(hatch none 0.1)
-		(priority 30006)
+		(priority 30003)
 		(attr
 			(teardrop
@@
 		(layer "B.Cu")
 		(hatch none 0.1)
-		(priority 30009)
+		(priority 30007)
 		(attr
 			(teardrop
@@
 		(layer "B.Cu")
 		(hatch none 0.1)
-		(priority 30010)
+		(priority 30009)
 		(attr
 			(teardrop
@@
 		(layer "B.Cu")
 		(hatch none 0.1)
-		(priority 30008)
+		(priority 30010)
 		(attr
 			(teardrop
@@
 		(layer "B.Cu")
 		(hatch none 0.1)
-		(priority 30007)
+		(priority 30008)
 		(attr
 			(teardrop

Commit message: details
Other:
- board text added: "mini"

Commit message: led names
Other:
- board text added: "10V+"
- board text added: "3v3+"
- board text added: "5v buck"
- board text added: "boot"
- board text added: "gyro"
- board text added: "status"

Commit message: Clean routing
Routing:
- net GND: track 84.7 -> 94.7 mm, vias 78 -> 182
- net /PADS/PIOUART0_TX: track 20.3 -> 14.7 mm
- net /PADS/LED_STRIP: track 53.4 -> 57.8 mm, vias 3 -> 5
- net /PADS/UART0_TX: track 13.6 -> 17.8 mm
- net /BLACKBOX/FLASH_CS: track 9.89 -> 13.7 mm
- net /PADS/U1RX: track 26.2 -> 29.3 mm
- net /POWER/10V_ENABLE: track 12.1 -> 14.9 mm
- net /PADS/UART0_RX: track 16.5 -> 14.1 mm
- net /PADS/M4: track 15.0 -> 12.5 mm, vias 1 -> 2
- net /BLACKBOX/SPI0.MOSI: track 8.15 -> 10.2 mm
- net /PADS/PU0RX: track 28.4 -> 30.1 mm
- net /PADS/M2: track 12.2 -> 10.8 mm, vias 1 -> 2
- net /PADS/M3: track 13.5 -> 12.4 mm, vias 1 -> 2
- net /RP2350A/LED0: track 12.5 -> 13.6 mm
- net /OSD/VIDEO_IN: track 5.90 -> 6.91 mm, vias 1 -> 2
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Other:
- board text added: "10V"
- board text removed: "10V+"
- board text removed: "3v3+"
