File: hardware/osd.kicad_sch (KiCad schematic)
At the start: 17 parts, among them U1 COS8051SOT, U18 SN74LVC1G3157DTBR, U2 TLV7031DPWR

Commit message: docs(schematic): add design annotations to all sheets
Port on-canvas engineering comments from OpenFC-Lite (RP2354B), adapted to the
Mini layout. +41 text items across root, rp2350a, power, imu, osd, blackbox,
pads. Annotation/text only — no net or connectivity changes. Mirrors
hardware/DESIGN_NOTES.md.

Co-Authored-By: Claude Opus 4.8 (1M context) <noreply@anthropic.com>
Other:
- note added: "06/06/2026"
- note added: "2"
- note added: "75R input terminatiom"
- note added: "Analog OSD using PIO State Machine on RP2350"
- note added: "Comparator detects sync pulses, read by RP2350 PIO"
- note added: "Resistor divider let's GPIO port select between high (VOH = 1V: white) or low (VOL = 0.3v: black)"

Commit message: chore(bom): consolidate LCSC Part -> LCSC field across schematic, library, footprints, project
Single canonical LCSC field (was split LCSC / LCSC Part). Every part resolves to one LCSC code; netlist verified, no duplicates. Includes Rev2 re-annotation resync re-save.

Co-Authored-By: Claude Opus 4.8 (1M context) <noreply@anthropic.com>
Parts:
- D9: LCSC (none) -> C151629; LCSC Part C151629 -> (none)
- U1: LCSC (none) -> C7463385; LCSC Part C7463385 -> (none)
- U18: LCSC (none) -> C2673087; LCSC Part C2673087 -> (none)
- U2: LCSC (none) -> C2876045; LCSC Part C2876045 -> (none)
Changed lines of the file:
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@@
 			)
 		)
-		(property "LCSC Part" "C2876045"
+		(property "LCSC" "C2876045"
 			(at 210.82 128.27 0)
 			(hide yes)
@@
 			)
 		)
-		(property "LCSC Part" "C2673087"
+		(property "LCSC" "C2673087"
 			(at 149.86 177.8 0)
 			(hide yes)
@@
 			)
 		)
-		(property "LCSC Part" "C151629"
+		(property "LCSC" "C151629"
 			(at 156.21 114.3 0)
 			(hide yes)
@@
 			)
 		)
-		(property "LCSC Part" "C7463385"
+		(property "LCSC" "C7463385"
 			(at 191.77 193.04 0)
 			(hide yes)

Commit message: schematics: complete Manufacturer/MPN coverage, trim stray whitespace
22 field fixes across blackbox, osd, power, rp2350a: Manufacturer backfilled
from the LCSC catalogue, trailing space trimmed from four XL-1005UGC MPNs.
pads.kicad_sch (uncommitted WIP) untouched. Part of the fab-agnostic BOM
standardisation for quoting outside JLCPCB.

kicad-skip reflowed the touched files; structural diff shows only property
changes, ERC identical (163 violations before and after).

Co-Authored-By: Claude Fable 5 <noreply@anthropic.com>
Parts:
- R46, R47: MPN (none) -> RC0201FR-07510RL; Manufacturer (none) -> YAGEO
